Commit message: Merged changes from Object Rearrangement fork. Fixed some bugs. Added some constraint features and test code.

File: data/test_assets/URDF/kuka_iiwa/model_free_base.urdf (robot description, URDF)
Before this commit: robot lbr_iiwa, 8 links, 7 joints
Links:
- link lbr_iiwa_link_7: geometry collision mesh filename=meshes/link_7.stl; visual mesh filename=meshes/link_7.stl
