Commit message: clang-tidy and clean-up fridge asset format

File: data/test_assets/urdf/fridge/fridge.urdf (robot description, URDF)
Before this commit: robot fridge, 4 links, 3 joints
Links:
- link body: geometry collision box size=0.029014 0.690834 1.91906; collision box size=0.643 0.03 1.89126
- link bottom_door: geometry collision box size=0.08 0.686 0.788; visual mesh filename=bottom_door.glb scale=1.0 1.0 1.0
- link top_door: geometry collision box size=0.097 0.712 1.103; visual mesh filename=top_door.glb scale=1.0 1.0 1.0
